File: eesa-solder.kicad_pcb (KiCad board)
At the start: 2 copper layers, 65.7 x 84.7 mm, 5 parts

Commit message: push to github
Parts:
- removed D2: LED, LED_THT:LED_D5.0mm
- removed R2: R, Resistor_THT:R_Axial_DIN0207_L6.3mm_D2.5mm_P7.62mm_Horizontal
- added SW1: SW_SPST, Button_Switch_THT:SW_Slide_SPDT_Straight_CK_OS102011MS2Q, F.Cu at (185.7, 102.5)
- moved R1 24.3 mm to (205.2, 105.3), turned to 90 degrees
- moved D1 20.2 mm to (196.2, 101.7), turned to 0 degrees
- moved BT1 2.74 mm to (194.6, 84.7)
Connections:
- D1 pad 2: Net-(BT1-+) -> Net-(D1-A)
Routing:
- net Net-(D1-A): track 0.00 -> 12.4 mm
- net Net-(BT1--): track 28.5 -> 17.4 mm
- net Net-(D2-K): track 6.02 -> 0.00 mm
- net Net-(D1-K): track 6.02 -> 10.6 mm
- net Net-(BT1-+): track 48.7 -> 50.6 mm
Other:
- outline, holes or cut-outs redrawn
- board text added: "ATTACK ON TITAN"
- board text added: "SURVEY CORPS"
- board text removed: "AOT"
